File: Patch_Panel.brd (EAGLE design)
At the start: 114.3 x 186.7 mm, 34 parts

Commit message: Removed 2-pin Connectors and RJ45 Pass-Through
Parts:
- removed U$25, U$26, U$27, U$28, U$29, U$30, U$31, U$32: MLX-2-PIN, MRDT-2015-General:MLX-2-PIN
- removed U$33, U$34: RJ45-8PTH, SparkFun-Connectors:RJ45-8
Connections:
- removed net N$1: U$33.1, U$34.1
- removed net N$2: U$33.2, U$34.2
- removed net N$3: U$33.3, U$34.3
- removed net N$4: U$33.4, U$34.4
- removed net N$5: U$33.5, U$34.5
- removed net N$6: U$33.6, U$34.6
- removed net N$7: U$33.7, U$34.7
- removed net N$8: U$33.8, U$34.8
- net 12V: no longer U$25.P$2, U$26.P$2, U$27.P$2, U$28.P$2, U$29.P$2, U$30.P$2, U$31.P$2, U$32.P$2
- net GND: no longer U$25.P$1, U$26.P$1, U$27.P$1, U$28.P$1, U$29.P$1, U$30.P$1, U$31.P$1, U$32.P$1
Routing:
- net 5V: track 0.00 -> 447.0 mm
- added copper zone on layer 16, net 12V
- removed copper zone on layer 16, net GND
Other:
- board size 114.3 x 186.7 mm -> 114.3 x 152.4 mm
- board text added: "12V"
- board text added: "5V"
- board text added: "GND"

Commit message: un-deleted brd file and re-added dxf
Parts:
- added U$25, U$26, U$27, U$28, U$29, U$30, U$31, U$32: MLX-2-PIN, MRDT-2015-General:MLX-2-PIN
- added U$33, U$34, U$37, U$38, U$39, U$40, U$41, U$42, U$43, U$44: H_20020618-M02HORIZ, MRDT-2015-PowerBoard:20020618-M02
- moved U$17 146.9 mm to (57.1, -40.6)
- moved U$19 146.9 mm to (57.1, -22.9)
- moved U$21 146.9 mm to (57.1, -5.08)
- moved U$23 146.9 mm to (57.1, -58.4)
- moved U$1 102.4 mm to (94.0, -5.08)
- moved U$3 102.4 mm to (94.0, -22.9)
- moved U$5 102.4 mm to (94.0, -40.6)
- moved U$7 102.4 mm to (94.0, -58.4)
Connections:
- new net MOCO_1: U$25.P$2, U$37.R1, U$37.R2
- new net MOCO_2: U$26.P$2, U$38.R1, U$38.R2
- new net MOCO_3: U$27.P$2, U$39.R1, U$39.R2
- new net MOCO_4: U$28.P$2, U$40.R1, U$40.R2
- new net MOCO_5: U$29.P$2, U$41.R1, U$41.R2
- new net MOCO_6: U$30.P$2, U$42.R1, U$42.R2
- new net MOCO_7: U$31.P$2, U$43.R1, U$43.R2
- new net MOCO_8: U$32.P$2, U$44.R1, U$44.R2
- net 12V: now also U$1.P$3, U$10.P$3, U$11.P$3, U$12.P$3, U$13.P$3, U$14.P$3, U$15.P$3, U$16.P$3, U$17.P$3, U$18.P$3, U$19.P$3, U$2.P$3, U$20.P$3, U$21.P$3, U$22.P$3, U$23.P$3, U$24.P$3, U$3.P$3, U$33.R1, U$33.R2, U$4.P$3, U$5.P$3, U$6.P$3, U$7.P$3, U$8.P$3, U$9.P$3; no longer U$1.P$2, U$10.P$2, U$11.P$2, U$12.P$2, U$13.P$2, U$14.P$2, U$15.P$2, U$16.P$2, U$17.P$2, U$18.P$2, U$19.P$2, U$2.P$2, U$20.P$2, U$21.P$2, U$22.P$2, U$23.P$2, U$24.P$2, U$3.P$2, U$4.P$2, U$5.P$2, U$6.P$2, U$7.P$2, U$8.P$2, U$9.P$2
- net 5V: now also U$1.P$2, U$10.P$2, U$11.P$2, U$12.P$2, U$13.P$2, U$14.P$2, U$15.P$2, U$16.P$2, U$17.P$2, U$18.P$2, U$19.P$2, U$2.P$2, U$20.P$2, U$21.P$2, U$22.P$2, U$23.P$2, U$24.P$2, U$3.P$2, U$34.R1, U$34.R2, U$4.P$2, U$5.P$2, U$6.P$2, U$7.P$2, U$8.P$2, U$9.P$2; no longer U$1.P$1, U$10.P$1, U$11.P$1, U$12.P$1, U$13.P$1, U$14.P$1, U$15.P$1, U$16.P$1, U$17.P$1, U$18.P$1, U$19.P$1, U$2.P$1, U$20.P$1, U$21.P$1, U$22.P$1, U$23.P$1, U$24.P$1, U$3.P$1, U$4.P$1, U$5.P$1, U$6.P$1, U$7.P$1, U$8.P$1, U$9.P$1
- net GND: now also U$1.P$1, U$10.P$1, U$11.P$1, U$12.P$1, U$13.P$1, U$14.P$1, U$15.P$1, U$16.P$1, U$17.P$1, U$18.P$1, U$19.P$1, U$2.P$1, U$20.P$1, U$21.P$1, U$22.P$1, U$23.P$1, U$24.P$1, U$25.P$1, U$26.P$1, U$27.P$1, U$28.P$1, U$29.P$1, U$3.P$1, U$30.P$1, U$31.P$1, U$32.P$1, U$33.L1, U$33.L2, U$34.L1, U$34.L2, U$37.L1, U$37.L2, U$38.L1, U$38.L2, U$39.L1, U$39.L2, U$4.P$1, U$40.L1, U$40.L2, U$41.L1, U$41.L2, U$42.L1, U$42.L2, U$43.L1, U$43.L2, U$44.L1, U$44.L2, U$5.P$1, U$6.P$1, U$7.P$1, U$8.P$1, U$9.P$1; no longer U$1.P$3, U$10.P$3, U$11.P$3, U$12.P$3, U$13.P$3, U$14.P$3, U$15.P$3, U$16.P$3, U$17.P$3, U$18.P$3, U$19.P$3, U$2.P$3, U$20.P$3, U$21.P$3, U$22.P$3, U$23.P$3, U$24.P$3, U$3.P$3, U$4.P$3, U$5.P$3, U$6.P$3, U$7.P$3, U$8.P$3, U$9.P$3
Routing:
- net 5V: track 447.0 -> 482.6 mm
- net MOCO_8: track 0.00 -> 28.2 mm
- net MOCO_7: track 0.00 -> 28.2 mm
- net MOCO_5: track 0.00 -> 28.2 mm
- net MOCO_3: track 0.00 -> 28.2 mm
- net MOCO_1: track 0.00 -> 28.2 mm
- net MOCO_4: track 0.00 -> 28.2 mm
- net MOCO_2: track 0.00 -> 28.2 mm
- net MOCO_6: track 0.00 -> 28.2 mm
Other:
- board size 114.3 x 152.4 mm -> 119.4 x 226.1 mm
- board text added: "V_MOT"
