File: Patch_Panel.brd (EAGLE design)
At the start: 128.3 x 222.2 mm, 43 parts, among them M1_IN APP_2POS_CONFIGMOCO_VERT, M1_OUT APP_2POS_CONFIGMOCO_VERT_DUMMY, M2_IN APP_2POS_CONFIGMOCO_VERT, M2_OUT APP_2POS_CONFIGMOCO_VERT_DUMMY, M3_IN APP_2POS_CONFIGMOCO_VERT, M3_OUT APP_2POS_CONFIGMOCO_VERT_DUMMY, M4_IN APP_2POS_CONFIGMOCO_VERT, M4_OUT APP_2POS_CONFIGMOCO_VERT_DUMMY, M5_IN APP_2POS_CONFIGMOCO_VERT, M5_OUT APP_2POS_CONFIGMOCO_VERT_DUMMY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

Commit message: added missing route
Routing:
- net 5V: track 525.2 -> 553.1 mm
Changed lines of the file:
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@@
 <wire x1="70.358" y1="24.13" x2="74.168" y2="27.94" width="3.81" layer="16"/>
 <wire x1="74.168" y1="27.94" x2="88.773" y2="27.94" width="3.81" layer="16"/>
-<wire x1="88.773" y1="12.7" x2="112.395" y2="12.7" width="0" layer="19" extent="1-1"/>
+<wire x1="88.773" y1="12.7" x2="88.9" y2="12.7" width="0.4064" layer="16"/>
+<wire x1="88.9" y1="36.322" x2="93.98" y2="31.242" width="3.81" layer="1"/>
+<wire x1="93.98" y1="31.242" x2="107.315" y2="31.242" width="3.81" layer="1"/>
+<wire x1="107.315" y1="31.242" x2="112.395" y2="36.322" width="3.81" layer="1"/>
+<wire x1="88.773" y1="36.322" x2="88.9" y2="36.322" width="0" layer="19" extent="1-16"/>
 </signal>
 <signal name="12V">
