File: PatchPanel_Hardware/PatchPanel_Hardware.kicad_pcb (KiCad board)
At the start: 2 copper layers, 158.2 x 75.7 mm, 35 parts

Commit message: update rev 2 library
Parts:
- Conn1, Conn10, Conn11, Conn12, Conn13, Conn14, Conn15, Conn2, Conn23, Conn24, Conn3, Conn4, Conn5, Conn6, Conn7, Conn9: footprint PatchPanel_Hardware:Vertical_Anderson_Triple_SidebySide -> MRDT_Connectors:Anderson_3_Vertical_Side_by_Side
- Conn16, Conn17, Conn18, Conn19, Conn20, Conn21, Conn22, Conn8: footprint PowerBoard_Hardware:Vertical_Anderson_Double_SidebySide -> MRDT_Connectors:Anderson_2_Vertical_Sidy_by_Side
- REF** (x4): value Drill_Hole_632 -> 6_32_Hole; footprint PowerBoard_Hardware:Drill_Hole_632 -> MRDT_Drill_Holes:6_32_Hole; moved to B.Cu
