File: PatchPanel_Hardware/PatchPanel_Hardware.sch (KiCad schematic (older format))
At the start: 58 parts

Commit message: Symbols named and packages assigned
Parts:
- Conn1, Conn10, Conn11, Conn12, Conn13, Conn14, Conn15, Conn18, Conn19, Conn2, Conn20, Conn21, Conn22, Conn3, Conn4, Conn5, Conn6, Conn7, Conn9: renamed from Conn?; footprint (none) -> PatchPanel_Hardware:Vertical_Anderson_Triple_SidebySide
- Conn16, Conn17, Conn8: renamed from Conn?; footprint (none) -> PowerBoard_Hardware:Vertical_Anderson_Double_SidebySide

Commit message: Placed Connectors & Routed Traces
Parts:
- added Conn23, Conn24: AndersonPP, PatchPanel_Hardware:Vertical_Anderson_Triple_SidebySide, symbol MRDT_Connectors:AndersonPP
- Conn18, Conn19, Conn20, Conn21, Conn22: footprint PatchPanel_Hardware:Vertical_Anderson_Triple_SidebySide -> PowerBoard_Hardware:Vertical_Anderson_Double_SidebySide
Connections:
- wire segments 124 -> 139

Commit message: update rev 2 library
Parts:
- Conn1, Conn10, Conn11, Conn12, Conn13, Conn14, Conn15, Conn2, Conn23, Conn24, Conn3, Conn4, Conn5, Conn6, Conn7, Conn9: footprint PatchPanel_Hardware:Vertical_Anderson_Triple_SidebySide -> MRDT_Connectors:Anderson_3_Vertical_Side_by_Side
- Conn16, Conn17, Conn18, Conn19, Conn20, Conn21, Conn22, Conn8: footprint PowerBoard_Hardware:Vertical_Anderson_Double_SidebySide -> MRDT_Connectors:Anderson_2_Vertical_Sidy_by_Side
