File: PatchPanel_Hardware/PatchPanel.sch (KiCad schematic (older format))
At the start: 59 parts, among them Q1 Q_PMOS_DGS, Q10 Q_PMOS_DGS, Q11 Q_PMOS_DGS, Q12 Q_PMOS_DGS, Q13 Q_PMOS_DGS, Q14 Q_PMOS_DGS, Q15 Q_PMOS_DGS, Q16 Q_PMOS_DGS, Q17 Q_PMOS_DGS, Q18 Q_PMOS_DGS, Q19 Q_PMOS_DGS, Q2 Q_PMOS_DGS, Q20 Q_PMOS_DGS, Q21 Q_PMOS_DGS, Q22 Q_PMOS_DGS, Q23 Q_PMOS_DGS, Q24 Q_PMOS_DGS, Q25 Q_PMOS_DGS, Q26 Q_PMOS_DGS, Q27 Q_PMOS_DGS, Q28 Q_PMOS_DGS, Q29 Q_PMOS_DGS, Q3 Q_PMOS_DGS, Q30 Q_PMOS_DGS, Q31 Q_PMOS_DGS, Q32 Q_PMOS_DGS, Q4 Q_PMOS_DGS, Q5 Q_PMOS_DGS, Q6 Q_PMOS_DGS, Q7 Q_PMOS_DGS, Q8 Q_PMOS_DGS, Q9 Q_PMOS_DGS

Commit message: board
Parts:
- Conn19: footprint MRDT_Connectors:Anderson_2_Vertical_Sidy_by_Side -> MRDT_Connectors:Anderson_3_Vertical_Side_by_Side
- Conn19: footprint (none) -> MRDT_Connectors:Anderson_3_Vertical_Side_by_Side
- D1, D2, D3, D4: footprint (none) -> LED_SMD:LED_0603_1608Metric_Pad1.05x0.95mm_HandSolder
- R1, R2, R3, R4: footprint (none) -> Resistor_SMD:R_0603_1608Metric_Pad1.05x0.95mm_HandSolder
Connections:
- net labels added: Vact, Vlog
Changed lines of the file:
@@
 F 0 "Conn19" H 4223 6847 60  0000 R CNN
 F 1 "AndersonPP" H 4223 6953 60  0000 R CNN
-F 2 "MRDT_Connectors:Anderson_2_Vertical_Sidy_by_Side" H 4100 6250 60  0001 C CNN
+F 2 "MRDT_Connectors:Anderson_3_Vertical_Side_by_Side" H 4100 6250 60  0001 C CNN
 F 3 "" H 4100 6250 60  0001 C CNN
 	1    4250 6800
@@
 F 0 "R1" H 10170 2396 50  0000 L CNN
 F 1 "R" H 10170 2305 50  0000 L CNN
-F 2 "" V 10030 2350 50  0001 C CNN
+F 2 "Resistor_SMD:R_0603_1608Metric_Pad1.05x0.95mm_HandSolder" V 10030 2350 50  0001 C CNN
 F 3 "~" H 10100 2350 50  0001 C CNN
 	1    10100 2350
@@
 F 0 "D1" V 10138 2583 50  0000 R CNN
 F 1 "LED" V 10047 2583 50  0000 R CNN
-F 2 "" H 10100 2700 50  0001 C CNN
+F 2 "LED_SMD:LED_0603_1608Metric_Pad1.05x0.95mm_HandSolder" H 10100 2700 50  0001 C CNN
 F 3 "~" H 10100 2700 50  0001 C CNN
 	1    10100 2700
@@
 F 0 "R2" H 10520 2396 50  0000 L CNN
 F 1 "R" H 10520 2305 50  0000 L CNN
-F 2 "" V 10380 2350 50  0001 C CNN
+F 2 "Resistor_SMD:R_0603_1608Metric_Pad1.05x0.95mm_HandSolder" V 10380 2350 50  0001 C CNN
 F 3 "~" H 10450 2350 50  0001 C CNN
 	1    10450 2350
@@
 F 0 "D2" V 10488 2583 50  0000 R CNN
 F 1 "LED" V 10397 2583 50  0000 R CNN
-F 2 "" H 10450 2700 50  0001 C CNN
+F 2 "LED_SMD:LED_0603_1608Metric_Pad1.05x0.95mm_HandSolder" H 10450 2700 50  0001 C CNN
 F 3 "~" H 10450 2700 50  0001 C CNN
 	1    10450 2700
@@
 F 0 "R3" H 10220 5046 50  0000 L CNN
 F 1 "R" H 10220 4955 50  0000 L CNN
-F 2 "" V 10080 5000 50  0001 C CNN
+F 2 "Resistor_SMD:R_0603_1608Metric_Pad1.05x0.95mm_HandSolder" V 10080 5000 50  0001 C CNN
 F 3 "~" H 10150 5000 50  0001 C CNN
 	1    10150 5000
@@
 F 0 "D3" V 10188 5233 50  0000 R CNN
 F 1 "LED" V 10097 5233 50  0000 R CNN
-F 2 "" H 10150 5350 50  0001 C CNN
+F 2 "LED_SMD:LED_0603_1608Metric_Pad1.05x0.95mm_HandSolder" H 10150 5350 50  0001 C CNN
 F 3 "~" H 10150 5350 50  0001 C CNN
 	1    10150 5350
@@
 F 0 "R4" H 10570 5046 50  0000 L CNN
 F 1 "R" H 10570 4955 50  0000 L CNN
-F 2 "" V 10430 5000 50  0001 C CNN
+F 2 "Resistor_SMD:R_0603_1608Metric_Pad1.05x0.95mm_HandSolder" V 10430 5000 50  0001 C CNN
 F 3 "~" H 10500 5000 50  0001 C CNN
 	1    10500 5000
@@
 F 0 "D4" V 10538 5233 50  0000 R CNN
 F 1 "LED" V 10447 5233 50  0000 R CNN
-F 2 "" H 10500 5350 50  0001 C CNN
+F 2 "LED_SMD:LED_0603_1608Metric_Pad1.05x0.95mm_HandSolder" H 10500 5350 50  0001 C CNN
 F 3 "~" H 10500 5350 50  0001 C CNN
 	1    10500 5350
@@
 F 0 "Conn19" H 11423 1197 60  0000 R CNN
 F 1 "AndersonPP" H 11423 1303 60  0000 R CNN
-F 2 "" H 11300 600 60  0001 C CNN
+F 2 "MRDT_Connectors:Anderson_3_Vertical_Side_by_Side" H 11300 600 60  0001 C CNN
 F 3 "" H 11300 600 60  0001 C CNN
 	3    11450 1150
@@
 F 0 "Conn19" H 11173 547 60  0000 R CNN
 F 1 "AndersonPP" H 11173 653 60  0000 R CNN
-F 2 "" H 11050 -50 60  0001 C CNN
+F 2 "MRDT_Connectors:Anderson_3_Vertical_Side_by_Side" H 11050 -50 60  0001 C CNN
 F 3 "" H 11050 -50 60  0001 C CNN
 	2    11200 500
@@
 $EndComp
 Connection ~ 10800 600
+Text Label 3850 5200 0    50   ~ 0
+GND
+Text Label 10550 600  0    50   ~ 0
+Vlog
+Text Label 10850 1250 0    50   ~ 0
+Vact
 $EndSCHEMATC
