File: PatchPanel_Hardware/PatchPanel.sch (KiCad schematic (older format))
At the start: 59 parts, among them Q1 Q_PMOS_DGS, Q10 Q_PMOS_DGS, Q11 Q_PMOS_DGS, Q12 Q_PMOS_DGS, Q13 Q_PMOS_DGS, Q14 Q_PMOS_DGS, Q15 Q_PMOS_DGS, Q16 Q_PMOS_DGS, Q17 Q_PMOS_DGS, Q18 Q_PMOS_DGS, Q19 Q_PMOS_DGS, Q2 Q_PMOS_DGS, Q20 Q_PMOS_DGS, Q21 Q_PMOS_DGS, Q22 Q_PMOS_DGS, Q23 Q_PMOS_DGS, Q24 Q_PMOS_DGS, Q25 Q_PMOS_DGS, Q26 Q_PMOS_DGS, Q27 Q_PMOS_DGS, Q28 Q_PMOS_DGS, Q29 Q_PMOS_DGS, Q3 Q_PMOS_DGS, Q30 Q_PMOS_DGS, Q31 Q_PMOS_DGS, Q32 Q_PMOS_DGS, Q4 Q_PMOS_DGS, Q5 Q_PMOS_DGS, Q6 Q_PMOS_DGS, Q7 Q_PMOS_DGS, Q8 Q_PMOS_DGS, Q9 Q_PMOS_DGS

Commit message: ready for board review
Parts:
- removed Conn18: Molex_SL_10, MRDT_Connectors:MOLEX_SL_10_Vertical, symbol MRDT_Connectors:Molex_SL_10
- removed unit 2 of Conn7
- removed unit 3 of Conn7
- removed D3, D4: LED, LED_SMD:LED_0603_1608Metric_Pad1.05x0.95mm_HandSolder, symbol Device:LED
- removed Q10, Q11, Q12, Q13, Q14, Q15, Q16, Q25, Q26, Q27, Q28, Q29, Q30, Q31, Q32, Q9: Q_PMOS_DGS, Package_TO_SOT_SMD:SOT-23, symbol Device:Q_PMOS_DGS
- added unit 2 of Conn9
- added unit 3 of Conn9
- added Q10, Q11, Q12, Q13, Q14, Q15, Q16, Q25, Q26, Q27, Q28, Q29, Q30, Q31, Q32, Q9: Q_NMOS_DGS, Package_TO_SOT_SMD:SOT-23, symbol Device:Q_NMOS_DGS
- added R1, R10, R11, R12, R13, R14, R15, R16, R17, R18, R19, R2, R20, R21, R22, R23, R24, R25, R26, R27, R28, R29, R30, R31, R32, R5, R6, R7, R8, R9: R, Resistor_SMD:R_0603_1608Metric_Pad1.05x0.95mm_HandSolder, symbol Device:R
- renumbered Conn19 to Conn1, Conn9 to Conn10, Conn19 to Conn18, Conn10 to Conn18, Conn1 to Conn7, Conn10 to Conn9, R1 to R33, R2 to R34
Connections:
- wire segments 269 -> 313
Other:
- note added: "12V Actuation\n"
- note added: "12V lgoic"
- note added: "GND"
- moved on the sheet: Conn10, Conn11A, Conn12A, Conn13A, Conn14A, Conn15A, Conn16A, Conn17A, Conn18A, Conn18B, Conn18C, Conn1A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

Commit message: final change
Parts:
- added Conn1: AndersonPP, MRDT_Connectors:Anderson_2_Vertical_Sidy_by_Side, symbol MRDT_Connectors:AndersonPP
- Conn1: footprint MRDT_Connectors:Anderson_3_Vertical_Side_by_Side -> MRDT_Connectors:Anderson_2_Vertical_Sidy_by_Side
Connections:
- wire segments 313 -> 314
Changed lines of the file:
@@
 F 0 "Conn1" H 906 6437 60  0000 C CNN
 F 1 "AndersonPP" H 906 6331 60  0000 C CNN
-F 2 "MRDT_Connectors:Anderson_3_Vertical_Side_by_Side" H 550 5500 60  0001 C CNN
+F 2 "MRDT_Connectors:Anderson_2_Vertical_Sidy_by_Side" H 550 5500 60  0001 C CNN
 F 3 "" H 550 5500 60  0001 C CNN
 	1    700  6050
@@
 Connection ~ 3600 7400
 Wire Wire Line
-	3600 7400 3600 6900
+	3600 7400 3600 7250
 Connection ~ 2000 7650
 Wire Wire Line
@@
 F 0 "Conn1" V 10650 1150 60  0000 R CNN
 F 1 "AndersonPP" V 10550 1250 60  0000 R CNN
-F 2 "MRDT_Connectors:Anderson_3_Vertical_Side_by_Side" H 10550 300 60  0001 C CNN
+F 2 "MRDT_Connectors:Anderson_2_Vertical_Sidy_by_Side" H 10550 300 60  0001 C CNN
 F 3 "" H 10550 300 60  0001 C CNN
 	3    10700 850
@@
 F 0 "Conn1" V 10350 700 60  0000 R CNN
 F 1 "AndersonPP" V 10423 753 60  0000 R CNN
-F 2 "MRDT_Connectors:Anderson_3_Vertical_Side_by_Side" H 10300 50  60  0001 C CNN
+F 2 "MRDT_Connectors:Anderson_2_Vertical_Sidy_by_Side" H 10300 50  60  0001 C CNN
 F 3 "" H 10300 50  60  0001 C CNN
 	2    10450 600
@@
 Wire Wire Line
 	11350 1850 11550 1850
+$Comp
+L MRDT_Connectors:AndersonPP Conn1
+U 1 1 5DD8D086
+P 4000 7150
+F 0 "Conn1" H 3973 7197 60  0000 R CNN
+F 1 "AndersonPP" H 3973 7303 60  0000 R CNN
+F 2 "MRDT_Connectors:Anderson_2_Vertical_Sidy_by_Side" H 3850 6600 60  0001 C CNN
+F 3 "" H 3850 6600 60  0001 C CNN
+	1    4000 7150
+	-1   0    0    1
+$EndComp
+Connection ~ 3600 7250
+Wire Wire Line
+	3600 7250 3600 6900
 $EndSCHEMATC

Commit message: before review
Parts:
- removed unit 3 of Conn1
- added unit 2 of Conn19
- renumbered Conn1 to Conn19
Changed lines of the file:
@@
-$Comp
-L MRDT_Connectors:AndersonPP Conn1
-U 3 1 5DA7FA5D
-P 10700 850
-F 0 "Conn1" V 10650 1150 60  0000 R CNN
-F 1 "AndersonPP" V 10550 1250 60  0000 R CNN
-F 2 "MRDT_Connectors:Anderson_2_Vertical_Sidy_by_Side" H 10550 300 60  0001 C CNN
-F 3 "" H 10550 300 60  0001 C CNN
-	3    10700 850
-	0    1    1    0
-$EndComp
 $Comp
 L MRDT_Connectors:AndersonPP Conn1
@@
 	11350 1850 11550 1850
 $Comp
-L MRDT_Connectors:AndersonPP Conn1
+L MRDT_Connectors:AndersonPP Conn19
 U 1 1 5DD8D086
 P 4000 7150
-F 0 "Conn1" H 3973 7197 60  0000 R CNN
+F 0 "Conn19" H 3973 7197 60  0000 R CNN
 F 1 "AndersonPP" H 3973 7303 60  0000 R CNN
 F 2 "MRDT_Connectors:Anderson_2_Vertical_Sidy_by_Side" H 3850 6600 60  0001 C CNN
@@
 Wire Wire Line
 	3600 7250 3600 6900
+$Comp
+L MRDT_Connectors:AndersonPP Conn19
+U 2 1 5DD8D04A
+P 10700 850
+F 0 "Conn19" V 10853 1078 60  0000 L CNN
+F 1 "AndersonPP" V 10959 1078 60  0000 L CNN
+F 2 "MRDT_Connectors:Anderson_2_Vertical_Sidy_by_Side" H 10550 300 60  0001 C CNN
+F 3 "" H 10550 300 60  0001 C CNN
+	2    10700 850
+	0    1    1    0
+$EndComp
 $EndSCHEMATC

Commit message: fixed board review issue
Parts:
- removed unit 2 of Conn19
- removed unit 2 of Conn9
- removed unit 3 of Conn9
- removed Q1, Q17, Q18, Q19, Q20, Q21, Q22, Q23, Q24, Q3, Q4, Q5, Q6, Q7, Q8: Q_PMOS_DGS, Package_TO_SOT_SMD:SOT-23, symbol Device:Q_PMOS_DGS
- removed Q13, Q14, Q25, Q29, Q30, Q9: Q_NMOS_DGS, Package_TO_SOT_SMD:SOT-23, symbol Device:Q_NMOS_DGS
- removed R1, R2, R25, R26: R, Resistor_SMD:R_0603_1608Metric_Pad1.05x0.95mm_HandSolder, symbol Device:R
- added unit 2 of Conn18
- added unit 2 of Conn3
- added unit 3 of Conn3
- added Q1, Q10, Q13, Q14, Q17, Q18, Q21, Q22, Q25, Q26, Q29, Q30, Q5, Q6, Q9: Q_PMOS_DGS, Package_TO_SOT_SMD:TO-252-2, symbol Device:Q_PMOS_GDS
- added Q19, Q20, Q23, Q24, Q7, Q8: Q_NMOS_DGS, Package_TO_SOT_SMD:SOT-323_SC-70_Handsoldering, symbol Device:Q_NMOS_DGS
- added R19, R20, R33, R34: 22k, Resistor_SMD:R_0603_1608Metric_Pad1.05x0.95mm_HandSolder, symbol Device:R
- Conn1: footprint MRDT_Connectors:Anderson_2_Vertical_Sidy_by_Side -> MRDT_Connectors:Anderson_3_Vertical_Side_by_Side
- Conn17: renamed from Conn19; footprint MRDT_Connectors:Anderson_2_Vertical_Sidy_by_Side -> MRDT_Connectors:Anderson_3_Vertical_Side_by_Side
- Conn18: footprint MRDT_Connectors:Anderson_3_Vertical_Side_by_Side -> MRDT_Connectors:Anderson_2_Vertical_Sidy_by_Side
- Conn9: renamed from Conn3; footprint MRDT_Connectors:Anderson_3_Vertical_Side_by_Side -> MRDT_Connectors:Anderson_2_Vertical_Sidy_by_Side
- Q11, Q12, Q15, Q16, Q27, Q28, Q31, Q32: footprint Package_TO_SOT_SMD:SOT-23 -> Package_TO_SOT_SMD:SOT-323_SC-70_Handsoldering
- Q2: footprint Package_TO_SOT_SMD:SOT-23 -> Package_TO_SOT_SMD:TO-252-2; symbol Device:Q_PMOS_DGS -> Device:Q_PMOS_GDS
- Q3: renamed from Q26; footprint Package_TO_SOT_SMD:SOT-23 -> Package_TO_SOT_SMD:SOT-323_SC-70_Handsoldering
- Q4: renamed from Q10; footprint Package_TO_SOT_SMD:SOT-23 -> Package_TO_SOT_SMD:SOT-323_SC-70_Handsoldering
- R1: renamed from R19; value R -> 22k
- R10, R11, R12, R13, R14, R15, R16, R17, R18, R21, R22, R23, R24, R27, R28, R29, R30, R31, R32, R4, R5, R6, R7, R8, R9: value R -> 22k
- R2: renamed from R3; value R -> 22k
- R3: renamed from R20; value R -> 22k
- renumbered Conn3 to Conn1, Conn7 to Conn10, Conn14 to Conn10, Conn11 to Conn10, Conn12 to Conn11, Conn13 to Conn11, Conn16 to Conn12, Conn13 to Conn12, Conn4 to Conn13, Conn14 to Conn13, Conn11 to Conn13, Conn8 to Conn14, Conn18 to Conn14, Conn15 to Conn14, Conn13 to Conn15, Conn17 to Conn15, Conn16 to Conn15, Conn17 to Conn16, Conn18 to Conn17, Conn15 to Conn17, Conn10 to Conn19, Conn5 to Conn2, Conn9 to Conn3, Conn14 to Conn4, Conn2 to Conn5, Conn11 to Conn7, Conn15 to Conn8, Conn1 to Conn9, R33 to R25, R34 to R26
Connections:
- net labels added: PF1, PF2, PF3, PG0, PL0, PL1, PL2, PL3, PL4, PL5
- wire segments 314 -> 300
Other:
- note added: "Act"
- note added: "All tiva control output\n"
- note added: "Always On Output"
- note added: "GND for all anderson\n"
- note added: "Logic"
- note added: "input power GND"
- note removed: "GND"
- moved on the sheet: Conn10A, Conn10B, Conn10C, Conn11A, Conn11B, Conn11C, Conn12A, Conn12B, Conn12C, Conn13A, Conn13B, Conn13C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

Commit message: change molex
Parts:
- Conn19: footprint MRDT_Connectors:MOLEX_SL_10_Vertical -> Connector_PinHeader_1.27mm:PinHeader_2x05_P1.27mm_Vertical
Changed lines of the file:
@@
 F 0 "Conn19" H 7644 6297 60  0000 C CNN
 F 1 "Molex_SL_10" H 7644 6191 60  0000 C CNN
-F 2 "MRDT_Connectors:MOLEX_SL_10_Vertical" H 7700 5600 60  0001 C CNN
+F 2 "Connector_PinHeader_1.27mm:PinHeader_2x05_P1.27mm_Vertical" H 7700 5600 60  0001 C CNN
 F 3 "" H 7700 5600 60  0001 C CNN
 	1    7700 5100
@@
 L power:GND #PWR08
 U 1 1 5DDF4403
-P 8050 2650
-F 0 "#PWR08" H 8050 2400 50  0001 C CNN
-F 1 "GND" H 8055 2477 50  0000 C CNN
-F 2 "" H 8050 2650 50  0001 C CNN
-F 3 "" H 8050 2650 50  0001 C CNN
-	1    8050 2650
-	1    0    0    -1
-$EndComp
+P 8050 2700
+F 0 "#PWR08" H 8050 2450 50  0001 C CNN
+F 1 "GND" H 8055 2527 50  0000 C CNN
+F 2 "" H 8050 2700 50  0001 C CNN
+F 3 "" H 8050 2700 50  0001 C CNN
+	1    8050 2700
+	1    0    0    -1
+$EndComp

Commit message: add LED to anderson
Parts:
- removed D1, D2: LED, LED_SMD:LED_0603_1608Metric_Pad1.05x0.95mm_HandSolder, symbol Device:LED
- removed R25, R26: R, Resistor_SMD:R_0603_1608Metric_Pad1.05x0.95mm_HandSolder, symbol Device:R
- added D10, D3, D4, D5, D6, D7, D8, D9: OrangeLED, LED_SMD:LED_0603_1608Metric_Pad1.05x0.95mm_HandSolder, symbol Device:LED
- added R35, R36, R37, R38, R39, R40, R41, R42: 300, Resistor_SMD:R_0603_1608Metric_Pad1.05x0.95mm_HandSolder, symbol Device:R
- Q1, Q10, Q13, Q14, Q17, Q18, Q2, Q21, Q22, Q25, Q26, Q29, Q30, Q5, Q6, Q9: value Q_PMOS_DGS -> Q_PMOS_GDS
- Q11, Q12, Q15, Q16, Q19, Q20, Q23, Q24, Q27, Q28, Q3, Q31, Q32, Q4, Q7, Q8: value Q_NMOS_DGS -> Q_NMOS_GSD; symbol Device:Q_NMOS_DGS -> Device:Q_NMOS_GSD
Connections:
- net labels removed: PF1, PF2
- wire segments 300 -> 318
Other:
- note added: "LED Indicator\n"

Commit message: BoardReview
Connections:
- net GND: now also Conn19.9
- net PF3 renamed PB8
- net PG0 renamed PB7
- net PL0 renamed PB4
- net PL1 renamed PB3
- net PL2 renamed PB2
- net PL3 renamed PB1
- net PL4 renamed PB6
- net PL5 renamed PB5
Other:
- note added: "PF3"
- note added: "PG0"
- note added: "PL0"
- note added: "PL1"
- note added: "PL2"
- note added: "PL3"
- note added: "PL4"
- note added: "PL5"
- moved on the sheet: D3, D4, D5, D6, D7, D8, R35, R36, R37, R38, R39, R40
