File: PatchPanel_Hardware/PatchPanel.kicad_pcb (KiCad board)
At the start: 2 copper layers, 52 parts, among them Q1 Q_PMOS_DGS, Q10 Q_PMOS_DGS, Q11 Q_PMOS_DGS, Q12 Q_PMOS_DGS, Q13 Q_PMOS_DGS, Q14 Q_PMOS_DGS, Q15 Q_PMOS_DGS, Q16 Q_PMOS_DGS, Q17 Q_PMOS_DGS, Q18 Q_PMOS_DGS, Q19 Q_PMOS_DGS, Q2 Q_PMOS_DGS, Q20 Q_PMOS_DGS, Q21 Q_PMOS_DGS, Q22 Q_PMOS_DGS, Q23 Q_PMOS_DGS, Q24 Q_PMOS_DGS, Q25 Q_PMOS_DGS, Q26 Q_PMOS_DGS, Q27 Q_PMOS_DGS, Q28 Q_PMOS_DGS, Q29 Q_PMOS_DGS, Q3 Q_PMOS_DGS, Q30 Q_PMOS_DGS, Q31 Q_PMOS_DGS, Q32 Q_PMOS_DGS, Q4 Q_PMOS_DGS, Q5 Q_PMOS_DGS, Q6 Q_PMOS_DGS, Q7 Q_PMOS_DGS, Q8 Q_PMOS_DGS, Q9 Q_PMOS_DGS, U6 Half_Booster_Mount

Commit message: board
Parts:
- removed U6: Half_Booster_Mount, MRDT_Shields:Half_Booster_Mount
- added D1: LED, LED_SMD:LED_0603_1608Metric_Pad1.05x0.95mm_HandSolder, F.Cu at (134.0, 62.2)
- added D2: LED, LED_SMD:LED_0603_1608Metric_Pad1.05x0.95mm_HandSolder, F.Cu at (134.0, 59.1)
- added D3: LED, LED_SMD:LED_0603_1608Metric_Pad1.05x0.95mm_HandSolder, F.Cu at (187.6, 62.2)
- added D4: LED, LED_SMD:LED_0603_1608Metric_Pad1.05x0.95mm_HandSolder, F.Cu at (187.6, 59.1)
- added R1: R, Resistor_SMD:R_0603_1608Metric_Pad1.05x0.95mm_HandSolder, F.Cu at (129.1, 62.2)
- added R2: R, Resistor_SMD:R_0603_1608Metric_Pad1.05x0.95mm_HandSolder, F.Cu at (129.1, 59.1)
- added R3: R, Resistor_SMD:R_0603_1608Metric_Pad1.05x0.95mm_HandSolder, F.Cu at (183.1, 62.2)
- added R4: R, Resistor_SMD:R_0603_1608Metric_Pad1.05x0.95mm_HandSolder, F.Cu at (183.1, 59.1)
- Conn19: footprint MRDT_Connectors:Anderson_2_Vertical_Sidy_by_Side -> MRDT_Connectors:Anderson_3_Vertical_Side_by_Side
- moved Conn17 176.3 mm to (225.1, 75.4)
- moved Conn16 157.0 mm to (214.3, 76.1)
- moved Conn15 137.5 mm to (203.2, 76.2)
- moved Conn12 122.0 mm to (171.1, 76.7)
- moved Conn14 118.4 mm to (192.4, 76.2)
- moved Q1 112.5 mm to (58.1, 69.9)
- moved Q2 107.2 mm to (70.2, 69.6)
- moved Q9 106.7 mm to (63.2, 69.8)
- moved Q3 102.7 mm to (81.6, 69.6)
- moved Conn11 102.1 mm to (159.7, 76.7)
- moved Q10 101.7 mm to (75.2, 69.6)
- moved Q11 96.1 mm to (86.7, 69.6)
- moved Q4 95.0 mm to (93.7, 69.6)
- moved Q5 90.1 mm to (105.1, 69.6)
- moved Conn13 89.8 mm to (181.9, 76.1)
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Connections:
- net Net-(Conn1-Pad1) renamed GND
- net Net-(Conn19-Pad2) renamed /Vlog
- Q10 pad 3: Net-(Conn19-Pad3) -> /Vact
- Q11 pad 3: Net-(Conn19-Pad3) -> /Vact
- Q12 pad 3: Net-(Conn19-Pad3) -> /Vact
- Q13 pad 3: Net-(Conn19-Pad3) -> /Vact
- Q14 pad 3: Net-(Conn19-Pad3) -> /Vact
- Q15 pad 3: Net-(Conn19-Pad3) -> /Vact
- Q16 pad 3: Net-(Conn19-Pad3) -> /Vact
- Q25 pad 3: Net-(Conn19-Pad3) -> /Vact
- Q26 pad 3: Net-(Conn19-Pad3) -> /Vact
- Q27 pad 3: Net-(Conn19-Pad3) -> /Vact
- Q28 pad 3: Net-(Conn19-Pad3) -> /Vact
- Q29 pad 3: Net-(Conn19-Pad3) -> /Vact
- Q30 pad 3: Net-(Conn19-Pad3) -> /Vact
- Q31 pad 3: Net-(Conn19-Pad3) -> /Vact
- Q32 pad 3: Net-(Conn19-Pad3) -> /Vact
- Q9 pad 3: Net-(Conn19-Pad3) -> /Vact
Routing:
- added copper zone on B.Cu, net GND
- added copper zone on F.Cu, net GND

Commit message: finished PCBdesign
Parts:
- moved D3 26.0 mm to (213.5, 59.9), turned to 180 degrees
- moved D4 26.0 mm to (213.5, 56.8), turned to 180 degrees
- moved R3 26.0 mm to (209.0, 59.9)
- moved R4 26.0 mm to (209.0, 56.8)
- moved Conn18 25.9 mm to (189.7, 58.8)
- moved Q32 5.29 mm to (231.6, 69.1)
- moved Q26 5.27 mm to (166.9, 69.6)
- moved Q23 5.02 mm to (215.6, 69.4)
- moved Q24 4.91 mm to (226.6, 69.1)
- moved Q31 4.83 mm to (220.4, 69.3)
- moved Q18 4.63 mm to (162.1, 69.6)
- moved Conn1 4.58 mm to (52.2, 76.4)
- moved Conn2 4.58 mm to (64.3, 76.4)
- moved Conn3 4.58 mm to (75.7, 76.4)
- moved Conn4 4.58 mm to (87.1, 76.4)
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Routing:
- net /Vlog: track 0.00 -> 251.4 mm, vias 0 -> 16
- net /Vact: track 0.00 -> 224.8 mm, vias 0 -> 16
- net Net-(Conn9-Pad1): track 0.00 -> 52.8 mm
- net Net-(Conn18-Pad8): track 0.00 -> 44.5 mm
- net Net-(Conn9-Pad2): track 0.00 -> 42.7 mm
- net Net-(Conn18-Pad1): track 0.00 -> 38.8 mm
- net Net-(Conn18-Pad7): track 0.00 -> 35.8 mm
- net Net-(Conn9-Pad3): track 0.00 -> 34.6 mm
- net Net-(Conn9-Pad8): track 0.00 -> 33.5 mm
- net Net-(Conn14-Pad3): track 0.00 -> 33.1 mm
- net Net-(Conn2-Pad3): track 0.00 -> 32.5 mm
- net Net-(Conn3-Pad3): track 0.00 -> 32.5 mm
- net Net-(Conn6-Pad3): track 0.00 -> 32.5 mm
- net Net-(Conn5-Pad3): track 0.00 -> 32.3 mm
- net Net-(Conn7-Pad3): track 0.00 -> 32.2 mm
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
Commit message: ready for board review
Parts:
- removed Conn19: AndersonPP, MRDT_Connectors:Anderson_3_Vertical_Side_by_Side
- removed D3, D4: LED, LED_SMD:LED_0603_1608Metric_Pad1.05x0.95mm_HandSolder
- added G***: LOGO, MRDT_Silkscreens:z_sig_SanfanLiu_sig21.8mmx12.3mm1, F.Cu at (95.9, 40.6)
- added G***: LOGO, MRDT_Silkscreens:0_MRDT_Logo_10mm, F.Cu at (48.9, 40.6)
- added R10: R, Resistor_SMD:R_0603_1608Metric_Pad1.05x0.95mm_HandSolder, F.Cu at (162.1, 52.5)
- added R11: R, Resistor_SMD:R_0603_1608Metric_Pad1.05x0.95mm_HandSolder, F.Cu at (73.9, 52.6)
- added R12: R, Resistor_SMD:R_0603_1608Metric_Pad1.05x0.95mm_HandSolder, F.Cu at (79.0, 52.6)
- added R13: R, Resistor_SMD:R_0603_1608Metric_Pad1.05x0.95mm_HandSolder, F.Cu at (199.4, 52.7)
- added R14: R, Resistor_SMD:R_0603_1608Metric_Pad1.05x0.95mm_HandSolder, F.Cu at (204.8, 52.7)
- added R15: R, Resistor_SMD:R_0603_1608Metric_Pad1.05x0.95mm_HandSolder, F.Cu at (95.1, 52.5)
- added R16: R, Resistor_SMD:R_0603_1608Metric_Pad1.05x0.95mm_HandSolder, F.Cu at (100.2, 52.5)
- added R17: R, Resistor_SMD:R_0603_1608Metric_Pad1.05x0.95mm_HandSolder, F.Cu at (167.7, 52.5)
- added R18: R, Resistor_SMD:R_0603_1608Metric_Pad1.05x0.95mm_HandSolder, F.Cu at (172.4, 52.7)
- added R19: R, Resistor_SMD:R_0603_1608Metric_Pad1.05x0.95mm_HandSolder, F.Cu at (41.7, 52.1)
- added R20: R, Resistor_SMD:R_0603_1608Metric_Pad1.05x0.95mm_HandSolder, F.Cu at (47.2, 52.0)
- added R21: R, Resistor_SMD:R_0603_1608Metric_Pad1.05x0.95mm_HandSolder, F.Cu at (105.3, 52.5)
- added R22: R, Resistor_SMD:R_0603_1608Metric_Pad1.05x0.95mm_HandSolder, F.Cu at (110.3, 52.5)
- added R23: R, Resistor_SMD:R_0603_1608Metric_Pad1.05x0.95mm_HandSolder, F.Cu at (125.9, 52.4)
- added R24: R, Resistor_SMD:R_0603_1608Metric_Pad1.05x0.95mm_HandSolder, F.Cu at (130.7, 52.4)
- added R25: R, Resistor_SMD:R_0603_1608Metric_Pad1.05x0.95mm_HandSolder, F.Cu at (146.2, 52.5)
- added R26: R, Resistor_SMD:R_0603_1608Metric_Pad1.05x0.95mm_HandSolder, F.Cu at (150.7, 52.5)
- added R27: R, Resistor_SMD:R_0603_1608Metric_Pad1.05x0.95mm_HandSolder, F.Cu at (63.8, 52.5)
- added R28: R, Resistor_SMD:R_0603_1608Metric_Pad1.05x0.95mm_HandSolder, F.Cu at (68.8, 52.5)
- added R29: R, Resistor_SMD:R_0603_1608Metric_Pad1.05x0.95mm_HandSolder, F.Cu at (188.8, 52.7)
- added R30: R, Resistor_SMD:R_0603_1608Metric_Pad1.05x0.95mm_HandSolder, F.Cu at (193.5, 52.7)
- added R31: R, Resistor_SMD:R_0603_1608Metric_Pad1.05x0.95mm_HandSolder, F.Cu at (84.3, 52.5)
- added R32: R, Resistor_SMD:R_0603_1608Metric_Pad1.05x0.95mm_HandSolder, F.Cu at (89.3, 52.5)
- added R33: R, Resistor_SMD:R_0603_1608Metric_Pad1.05x0.95mm_HandSolder, F.Cu at (150.5, 37.4)
- added R34: R, Resistor_SMD:R_0603_1608Metric_Pad1.05x0.95mm_HandSolder, F.Cu at (150.5, 40.2)
- added R5: R, Resistor_SMD:R_0603_1608Metric_Pad1.05x0.95mm_HandSolder, F.Cu at (115.7, 52.3)
- added R6: R, Resistor_SMD:R_0603_1608Metric_Pad1.05x0.95mm_HandSolder, F.Cu at (120.7, 52.4)
- added R7: R, Resistor_SMD:R_0603_1608Metric_Pad1.05x0.95mm_HandSolder, F.Cu at (136.3, 52.4)
- added R8: R, Resistor_SMD:R_0603_1608Metric_Pad1.05x0.95mm_HandSolder, F.Cu at (140.7, 52.4)
- added R9: R, Resistor_SMD:R_0603_1608Metric_Pad1.05x0.95mm_HandSolder, F.Cu at (156.6, 52.5)
- Conn10: value AndersonPP -> Molex_SL_10; footprint MRDT_Connectors:Anderson_3_Vertical_Side_by_Side -> MRDT_Connectors:MOLEX_SL_10_Vertical
- Conn18, Conn9: value Molex_SL_10 -> AndersonPP; footprint MRDT_Connectors:MOLEX_SL_10_Vertical -> MRDT_Connectors:Anderson_3_Vertical_Side_by_Side
- Q10, Q11, Q12, Q13, Q14, Q15, Q16, Q25, Q26, Q27, Q28, Q29, Q30, Q31, Q32, Q9: value Q_PMOS_DGS -> Q_NMOS_DGS
- moved R3 156.6 mm to (52.7, 52.3), turned to 180 degrees
- moved R4 151.1 mm to (58.0, 52.3), turned to 180 degrees
- moved Q32 144.1 mm to (89.2, 47.7), turned to 180 degrees
- moved Q24 143.8 mm to (84.3, 47.8), turned to 90 degrees
- moved Q30 142.7 mm to (68.8, 47.8), turned to 180 degrees
- moved Q22 142.6 mm to (63.8, 47.8), turned to 90 degrees
- moved Q18 122.4 mm to (41.7, 47.8), turned to 90 degrees
- moved Q1 122.3 mm to (178.3, 47.6), turned to 90 degrees
- moved Q26 121.8 mm to (47.1, 47.7), turned to 180 degrees
- moved Q9 121.7 mm to (182.9, 47.6), turned to 180 degrees
- moved Conn14 121.2 mm to (75.8, 109.3), turned to 90 degrees
- moved Conn2 116.5 mm to (180.7, 81.0), turned to 90 degrees
- moved Conn12 115.8 mm to (60.0, 109.3), turned to 90 degrees
- moved Conn17 93.3 mm to (138.2, 109.3), turned to 90 degrees
- moved Conn13 91.5 mm to (96.6, 109.3), turned to 90 degrees
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Connections:
- Conn1 pad 2: Net-(Conn1-Pad2) -> /Vlog
- Conn1 pad 3: Net-(Conn1-Pad3) -> /Vact
- Conn10 pad 1: GND -> Net-(Conn10-Pad1)
- Conn11 pad 2: Net-(Conn11-Pad2) -> /Vlog
- Conn11 pad 3: Net-(Conn11-Pad3) -> /Vact
- Conn12 pad 2: Net-(Conn12-Pad2) -> /Vlog
- Conn12 pad 3: Net-(Conn12-Pad3) -> /Vact
- Conn13 pad 2: Net-(Conn13-Pad2) -> /Vlog
- Conn13 pad 3: Net-(Conn13-Pad3) -> /Vact
- Conn14 pad 2: Net-(Conn14-Pad2) -> /Vlog
- Conn14 pad 3: Net-(Conn14-Pad3) -> /Vact
- Conn15 pad 2: Net-(Conn15-Pad2) -> /Vlog
- Conn15 pad 3: Net-(Conn15-Pad3) -> /Vact
- Conn16 pad 2: Net-(Conn16-Pad2) -> /Vlog
- Conn16 pad 3: Net-(Conn16-Pad3) -> /Vact
- Conn17 pad 2: Net-(Conn17-Pad2) -> /Vlog
- Conn17 pad 3: Net-(Conn17-Pad3) -> /Vact
- Conn18 pad 1: Net-(Conn18-Pad1) -> GND
- Conn18 pad 2: Net-(Conn18-Pad2) -> /Vlog
- Conn18 pad 3: Net-(Conn18-Pad3) -> /Vact
- Conn9 pad 1: Net-(Conn9-Pad1) -> GND
- Q1 pad 1: Net-(Conn1-Pad2) -> /Vlog
- Q1 pad 2: Net-(Conn9-Pad1) -> Net-(Q1-Pad2)
- Q1 pad 3: /Vlog -> Net-(Conn2-Pad2)
- Q10 pad 1: Net-(Conn2-Pad3) -> Net-(Q10-Pad1)
- Q10 pad 2: Net-(Conn9-Pad2) -> Net-(Conn10-Pad1)
- Q10 pad 3: /Vact -> GND
- Q11 pad 1: Net-(Conn3-Pad3) -> Net-(Q11-Pad1)
- Q11 pad 2: Net-(Conn9-Pad3) -> Net-(Conn10-Pad4)
- Q11 pad 3: /Vact -> GND
- Q12 pad 1: Net-(Conn4-Pad3) -> Net-(Q12-Pad1)
- Q12 pad 2: Net-(Conn9-Pad4) -> Net-(Conn10-Pad5)
- Q12 pad 3: /Vact -> GND
- Q13 pad 1: Net-(Conn5-Pad3) -> Net-(Q13-Pad1)
- Q13 pad 2: Net-(Conn9-Pad5) -> Net-(Conn10-Pad6)
- Q13 pad 3: /Vact -> GND
- Q14 pad 1: Net-(Conn6-Pad3) -> Net-(Q14-Pad1)
- Q14 pad 2: Net-(Conn9-Pad6) -> Net-(Conn10-Pad2)
- Q14 pad 3: /Vact -> GND
- Q15 pad 1: Net-(Conn7-Pad3) -> Net-(Q15-Pad1)
- Q15 pad 2: Net-(Conn9-Pad7) -> Net-(Conn10-Pad8)
- Q15 pad 3: /Vact -> GND
- Q16 pad 1: Net-(Conn8-Pad3) -> Net-(Q16-Pad1)
- Q16 pad 2: Net-(Conn9-Pad8) -> Net-(Conn10-Pad3)
- Q16 pad 3: /Vact -> GND
- Q17 pad 1: Net-(Conn10-Pad2) -> /Vact
- Q17 pad 2: Net-(Conn18-Pad1) -> Net-(Q17-Pad2)
- Q17 pad 3: /Vlog -> Net-(Conn2-Pad3)
- Q18 pad 1: Net-(Conn11-Pad2) -> /Vact
- Q18 pad 2: Net-(Conn18-Pad2) -> Net-(Q18-Pad2)
- Q18 pad 3: /Vlog -> Net-(Conn3-Pad3)
- Q19 pad 1: Net-(Conn12-Pad2) -> /Vact
- Q19 pad 2: Net-(Conn18-Pad3) -> Net-(Q19-Pad2)
- Q19 pad 3: /Vlog -> Net-(Conn4-Pad3)
- Q2 pad 1: Net-(Conn2-Pad2) -> /Vlog
- Q2 pad 2: Net-(Conn9-Pad2) -> Net-(Q2-Pad2)
- Q2 pad 3: /Vlog -> Net-(Conn3-Pad2)
- Q20 pad 1: Net-(Conn13-Pad2) -> /Vact
- Q20 pad 2: Net-(Conn18-Pad4) -> Net-(Q20-Pad2)
- Q20 pad 3: /Vlog -> Net-(Conn5-Pad3)
- Q21 pad 1: Net-(Conn14-Pad2) -> /Vact
- Q21 pad 2: Net-(Conn18-Pad5) -> Net-(Q21-Pad2)
- Q21 pad 3: /Vlog -> Net-(Conn6-Pad3)
- Q22 pad 1: Net-(Conn15-Pad2) -> /Vact
- Q22 pad 2: Net-(Conn18-Pad6) -> Net-(Q22-Pad2)
- Q22 pad 3: /Vlog -> Net-(Conn7-Pad3)
- Q23 pad 1: Net-(Conn16-Pad2) -> /Vact
- Q23 pad 2: Net-(Conn18-Pad7) -> Net-(Q23-Pad2)
- Q23 pad 3: /Vlog -> Net-(Conn8-Pad3)
- Q24 pad 1: Net-(Conn17-Pad2) -> /Vact
- Q24 pad 2: Net-(Conn18-Pad8) -> Net-(Q24-Pad2)
- Q24 pad 3: /Vlog -> Net-(Conn9-Pad3)
- Q25 pad 1: Net-(Conn10-Pad3) -> Net-(Q25-Pad1)
- Q25 pad 2: Net-(Conn18-Pad1) -> Net-(Conn10-Pad7)
- Q25 pad 3: /Vact -> GND
- Q26 pad 1: Net-(Conn11-Pad3) -> Net-(Q26-Pad1)
- Q26 pad 2: Net-(Conn18-Pad2) -> Net-(Conn10-Pad1)
- Q26 pad 3: /Vact -> GND
- Q27 pad 1: Net-(Conn12-Pad3) -> Net-(Q27-Pad1)
- Q27 pad 2: Net-(Conn18-Pad3) -> Net-(Conn10-Pad4)
- Q27 pad 3: /Vact -> GND
- Q28 pad 1: Net-(Conn13-Pad3) -> Net-(Q28-Pad1)
- Q28 pad 2: Net-(Conn18-Pad4) -> Net-(Conn10-Pad5)
- Q28 pad 3: /Vact -> GND
- Q29 pad 1: Net-(Conn14-Pad3) -> Net-(Q29-Pad1)
- Q29 pad 2: Net-(Conn18-Pad5) -> Net-(Conn10-Pad6)
- Q29 pad 3: /Vact -> GND
- Q3 pad 1: Net-(Conn3-Pad2) -> /Vlog
- Q3 pad 2: Net-(Conn9-Pad3) -> Net-(Q3-Pad2)
- Q3 pad 3: /Vlog -> Net-(Conn4-Pad2)
- Q30 pad 1: Net-(Conn15-Pad3) -> Net-(Q30-Pad1)
- Q30 pad 2: Net-(Conn18-Pad6) -> Net-(Conn10-Pad2)
- Q30 pad 3: /Vact -> GND
- Q31 pad 1: Net-(Conn16-Pad3) -> Net-(Q31-Pad1)
- Q31 pad 2: Net-(Conn18-Pad7) -> Net-(Conn10-Pad8)
- Q31 pad 3: /Vact -> GND
- Q32 pad 1: Net-(Conn17-Pad3) -> Net-(Q32-Pad1)
- Q32 pad 2: Net-(Conn18-Pad8) -> Net-(Conn10-Pad3)
- Q32 pad 3: /Vact -> GND
- Q4 pad 1: Net-(Conn4-Pad2) -> /Vlog
- Q4 pad 2: Net-(Conn9-Pad4) -> Net-(Q4-Pad2)
- Q4 pad 3: /Vlog -> Net-(Conn5-Pad2)
- Q5 pad 1: Net-(Conn5-Pad2) -> /Vlog
- Q5 pad 2: Net-(Conn9-Pad5) -> Net-(Q5-Pad2)
- Q5 pad 3: /Vlog -> Net-(Conn6-Pad2)
- Q6 pad 1: Net-(Conn6-Pad2) -> /Vlog
- Q6 pad 2: Net-(Conn9-Pad6) -> Net-(Q6-Pad2)
- Q6 pad 3: /Vlog -> Net-(Conn7-Pad2)
- Q7 pad 1: Net-(Conn7-Pad2) -> /Vlog
- Q7 pad 2: Net-(Conn9-Pad7) -> Net-(Q7-Pad2)
- Q7 pad 3: /Vlog -> Net-(Conn8-Pad2)
- Q8 pad 1: Net-(Conn8-Pad2) -> /Vlog
- Q8 pad 2: Net-(Conn9-Pad8) -> Net-(Q8-Pad2)
- Q8 pad 3: /Vlog -> Net-(Conn9-Pad2)
- Q9 pad 1: Net-(Conn1-Pad3) -> Net-(Q9-Pad1)
- Q9 pad 2: Net-(Conn9-Pad1) -> Net-(Conn10-Pad7)
- Q9 pad 3: /Vact -> GND
- R1 pad 1: Net-(Conn9-Pad9) -> Net-(Q1-Pad2)
- R1 pad 2: Net-(D1-Pad2) -> /Vlog
- R2 pad 1: Net-(Conn9-Pad10) -> Net-(Q9-Pad1)
- R2 pad 2: Net-(D2-Pad2) -> Net-(Q1-Pad2)
- R3 pad 1: Net-(Conn18-Pad9) -> Net-(Q2-Pad2)
- R3 pad 2: Net-(D3-Pad2) -> /Vlog
- R4 pad 1: Net-(Conn18-Pad10) -> Net-(Q10-Pad1)
- R4 pad 2: Net-(D4-Pad2) -> Net-(Q2-Pad2)
Routing:
- net /Vact: track 224.8 -> 458.3 mm, vias 16 -> 8
- net /Vlog: track 251.4 -> 468.8 mm, vias 16 -> 8
- net Net-(Conn10-Pad8): track 0.00 -> 78.4 mm
- net Net-(Conn10-Pad1): track 0.00 -> 76.1 mm
- net Net-(Conn10-Pad7): track 0.00 -> 59.2 mm
- net Net-(Conn9-Pad1): track 52.8 -> 0.00 mm
- net Net-(Conn18-Pad8): track 44.5 -> 0.00 mm
- net Net-(Conn10-Pad6): track 0.00 -> 40.7 mm
- net Net-(Conn18-Pad1): track 38.8 -> 0.00 mm
- net Net-(Conn18-Pad7): track 35.8 -> 0.00 mm
- net Net-(Conn9-Pad8): track 33.5 -> 0.00 mm
- net Net-(Conn14-Pad3): track 33.1 -> 0.00 mm
- net Net-(Conn10-Pad2): track 24.3 -> 57.3 mm
- net Net-(Conn1-Pad3): track 31.6 -> 0.00 mm
- net Net-(Conn16-Pad3): track 31.6 -> 0.00 mm
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Other:
- board outline added: 172.1 x 75.6 mm
- board text added: "Patch Panel, Rev. 1 Mars Rover Design Team Missouri S&T, 2019 Sanfan Liu"

Commit message: add input label
Other:
- board text added: "Input"
Changed lines of the file:
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@@
   (general
     (thickness 1.6)
-    (drawings 5)
+    (drawings 6)
     (tracks 432)
     (zones 0)
@@
   )
   (setup
-    (last_trace_width 0.762)
+    (last_trace_width 0.25)
     (user_trace_width 0.381)
     (user_trace_width 0.762)
@@
     )
   )
+  (gr_text Input (at 40.64 83.82) (layer F.SilkS)
+    (effects (font (size 1.5 1.5) (thickness 0.3)))
+  )
   (gr_line (start 34.925 110.49) (end 34.925 34.925) (layer Edge.Cuts) (width 0.15))

Commit message: final change
Parts:
- added Conn19: AndersonPP, MRDT_Connectors:Anderson_2_Vertical_Sidy_by_Side, F.Cu at (46.1, 109.4)
- Conn1: footprint MRDT_Connectors:Anderson_3_Vertical_Side_by_Side -> MRDT_Connectors:Anderson_2_Vertical_Sidy_by_Side
- moved Conn1 44.8 mm to (37.7, 65.3), turned to 270 degrees
Connections:
- Conn1 pad 2: /Vlog -> (no net)
Routing:
- net /Vlog: track 468.8 -> 410.6 mm
- net /Vact: track 458.3 -> 411.0 mm

Commit message: before review
Parts:
- moved Conn1 45.2 mm to (46.1, 109.6), turned to 90 degrees
- moved Conn19 44.8 mm to (38.4, 65.3), turned to 270 degrees
Connections:
- Conn1 pad 2: (no net) -> /Vlog
- Conn19 pad 2: /Vlog -> /Vact
Routing:
- net /Vact: track 411.0 -> 433.3 mm
Changed lines of the file:
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@@
     (thickness 1.6)
     (drawings 6)
-    (tracks 425)
+    (tracks 428)
     (zones 0)
     (modules 89)
@@
   )
   (module MRDT_Connectors:Anderson_2_Vertical_Sidy_by_Side (layer F.Cu)
-    (at 37.745 65.265 270)
-    (fp_text reference Conn1 (at 13.7 1.6 270) (layer F.SilkS)
+    (at 46.075 109.64 90)
+    (fp_text reference Conn1 (at 13.7 1.6 90) (layer F.SilkS)
       (effects (font (size 1 1) (thickness 0.15)))
     )
-    (fp_text value AndersonPP (at 8.2 -9.2 90) (layer F.Fab) hide
+    (fp_text value AndersonPP (at 8.2 -9.2 270) (layer F.Fab) hide
       (effects (font (size 1 1) (thickness 0.15)))
     )
@@
     (fp_line (start 7.9 -7.9) (end 0 -7.9) (layer F.SilkS) (width 0.15))
     (fp_line (start 7.9 0) (end 0 0) (layer F.SilkS) (width 0.15))
-    (pad 2 thru_hole circle (at 11.85 -4.8 180) (size 5.08 5.08) (drill 4.104006) (layers *.Cu *.Mask))
-    (pad 1 thru_hole circle (at 3.95 -4.8 180) (size 5.08 5.08) (drill 4.104006) (layers *.Cu *.Mask)
+    (pad 2 thru_hole circle (at 11.85 -4.8) (size 5.08 5.08) (drill 4.104006) (layers *.Cu *.Mask)
+      (net 20 /Vlog))
+    (pad 1 thru_hole circle (at 3.95 -4.8) (size 5.08 5.08) (drill 4.104006) (layers *.Cu *.Mask)
       (net 19 GND))
     (model "${MRDT_KICAD_LIBRARIES}/3D Files/MRDT_Connctors/Anderson_2_Vertcal_Side_by_Side.stp"
@@
   )
   (module MRDT_Connectors:Anderson_2_Vertical_Sidy_by_Side (layer F.Cu)
-    (at 46.075 109.36 90)
-    (fp_text reference Conn19 (at 13.7 1.6 90) (layer F.SilkS)
+    (at 38.38 65.265 270)
+    (fp_text reference Conn19 (at 13.7 1.6 270) (layer F.SilkS)
       (effects (font (size 1 1) (thickness 0.15)))
     )
-    (fp_text value AndersonPP (at 8.2 -9.2 270) (layer F.Fab) hide
+    (fp_text value AndersonPP (at 8.2 -9.2 90) (layer F.Fab) hide
       (effects (font (size 1 1) (thickness 0.15)))
     )
@@
     (fp_line (start 15.8 0) (end 15.8 -7.9) (layer F.SilkS) (width 0.15))
     (fp_line (start 15.292 -6.35) (end 15.292 -1.778) (layer F.SilkS) (width 0.15))
-    (pad 1 thru_hole circle (at 3.95 -4.8) (size 5.08 5.08) (drill 4.104006) (layers *.Cu *.Mask)
+    (pad 1 thru_hole circle (at 3.95 -4.8 180) (size 5.08 5.08) (drill 4.104006) (layers *.Cu *.Mask)
       (net 19 GND))
-    (pad 2 thru_hole circle (at 11.85 -4.8) (size 5.08 5.08) (drill 4.104006) (layers *.Cu *.Mask)
-      (net 20 /Vlog))
+    (pad 2 thru_hole circle (at 11.85 -4.8 180) (size 5.08 5.08) (drill 4.104006) (layers *.Cu *.Mask)
+      (net 21 /Vact))
     (model "${MRDT_KICAD_LIBRARIES}/3D Files/MRDT_Connctors/Anderson_2_Vertcal_Side_by_Side.stp"
       (offset (xyz 15.87499976158142 6.984999895095826 0))
@@
     )
   )
-  (gr_text Input (at 40.64 83.82) (layer F.SilkS)
+  (gr_text Input (at 41.275 92.075) (layer F.SilkS)
     (effects (font (size 1.5 1.5) (thickness 0.3)))
   )
@@
   (segment (start 145.3134 55.9816) (end 144.78 56.515) (width 0.762) (layer F.Cu) (net 21))
   (segment (start 145.3134 52.5272) (end 145.3134 55.9816) (width 0.762) (layer F.Cu) (net 21))
+  (segment (start 55.2196 89.535) (end 46.99 89.535) (width 5) (layer B.Cu) (net 21))
+  (segment (start 43.18 85.725) (end 43.18 77.115) (width 5) (layer B.Cu) (net 21))
+  (segment (start 46.99 89.535) (end 43.18 85.725) (width 5) (layer B.Cu) (net 21))
   (segment (start 151.3446 37.3634) (end 154.0764 37.3634) (width 0.381) (layer F.Cu) (net 22))
   (segment (start 151.384 40.1574) (end 154.1158 40.1574) (width 0.381) (layer F.Cu) (net 23))
